File: electronics/test/Test.kicad_pcb (KiCad board)
At the start: 2 copper layers, 50.8 x 25.4 mm, 3 parts

Commit message: finished tutorial
Parts:
- moved R1 9.16 mm to (141.0, 78.7)
- moved D1 8.03 mm to (111.8, 78.7)
Routing:
- net /led: track 25.2 -> 14.0 mm
- net GND: track 10.7 -> 15.5 mm
- net VCC: track 16.3 -> 16.0 mm, vias 0 -> 1
- added copper zone on B.Cu, net GND
- added copper zone on F.Cu, net VCC
Other:
- board size 50.8 x 25.4 mm -> 50.8 x 33 mm
Changed lines of the file:
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@@
   (net 3 "/led")
   (footprint "Resistor_THT:R_Axial_DIN0309_L9.0mm_D3.2mm_P12.70mm_Horizontal" (layer "F.Cu")
-    (at 148.59 73.66 180)
+    (at 140.97 78.74 180)
     (descr "Resistor, Axial_DIN0309 series, Axial, Horizontal, pin pitch=12.7mm, 0.5W = 1/2W, length*diameter=9*3.2mm^2, http://cdn-reichelt.de/documents/datenblatt/B400/1_4W%23YAG.pdf")
     (tags "Resistor Axial_DIN0309 series Axial Horizontal pin pitch 12.7mm 0.5W = 1/2W length 9mm diameter 3.2mm")
@@
   )
   (footprint "LED_THT:LED_D5.0mm" (layer "F.Cu")
-    (at 109.22 71.12)
+    (at 111.76 78.74)
     (descr "LED, diameter 5.0mm, 2 pins, http://cdn-reichelt.de/documents/datenblatt/A500/LL-504BC2E-009.pdf")
     (tags "LED diameter 5.0mm 2 pins")
@@
     )
   )
-  (gr_rect (start 101.6 50.8) (end 152.4 76.2)
+  (gr_rect (start 101.6 50.8) (end 152.4 83.82)
     (stroke (width 0.1) (type default)) (fill none) (layer "Edge.Cuts"))
-  (segment (start 141.68 63.5) (end 147.32 63.5) (width 0.25) (layer "B.Cu") (net 1))
-  (segment (start 147.32 63.5) (end 148.59 64.77) (width 0.25) (layer "B.Cu") (net 1))
-  (segment (start 148.59 64.77) (end 148.59 73.66) (width 0.25) (layer "B.Cu") (net 1))
-  (segment (start 109.22 63.5) (end 109.22 71.12) (width 0.25) (layer "B.Cu") (net 2))
-  (segment (start 112.32 63.5) (end 109.22 63.5) (width 0.25) (layer "B.Cu") (net 2))
-  (segment (start 133.35 71.12) (end 135.89 73.66) (width 0.25) (layer "F.Cu") (net 3))
-  (segment (start 111.76 71.12) (end 133.35 71.12) (width 0.25) (layer "F.Cu") (net 3))
+  (segment (start 142.24 71.12) (end 140.97 72.39) (width 0.25) (layer "F.Cu") (net 1))
+  (segment (start 140.97 72.39) (end 140.97 78.74) (width 0.25) (layer "F.Cu") (net 1))
+  (via (at 142.24 71.12) (size 0.8) (drill 0.4) (layers "F.Cu" "B.Cu") (net 1))
+  (segment (start 141.68 70.56) (end 142.24 71.12) (width 0.25) (layer "B.Cu") (net 1))
+  (segment (start 141.68 63.5) (end 141.68 70.56) (width 0.25) (layer "B.Cu") (net 1))
+  (segment (start 112.32 78.18) (end 111.76 78.74) (width 0.25) (layer "B.Cu") (net 2))
+  (segment (start 112.32 63.5) (end 112.32 78.18) (width 0.25) (layer "B.Cu") (net 2))
+  (segment (start 114.3 78.74) (end 128.27 78.74) (width 0.25) (layer "F.Cu") (net 3))
+  (zone (net 1) (net_name "VCC") (layer "F.Cu") (hatch edge 0.5)
+    (priority 1)
+    (connect_pads (clearance 0.5))
+    (min_thickness 0.25) (filled_areas_thickness no)
+    (fill yes (thermal_gap 0.5) (thermal_bridge_width 0.5))
+    (polygon
+      (pts
+        (xy 101.6 50.8)
+        (xy 101.6 83.82)
+        (xy 152.4 83.82)
+        (xy 152.4 50.8)
+      )
+    )
+  )
+  (zone (net 2) (net_name "GND") (layer "B.Cu") (hatch edge 0.5)
+    (connect_pads (clearance 0.5))
+    (min_thickness 0.25) (filled_areas_thickness no)
+    (fill yes (thermal_gap 0.5) (thermal_bridge_width 0.5))
+    (polygon
+      (pts
+        (xy 101.6 50.8)
+        (xy 152.4 50.8)
+        (xy 152.4 83.82)
+        (xy 101.6 83.82)
+        (xy 101.6 63.5)
+      )
+    )
+  )
 )
