File: electronics/fluke-8200a-power-supply/fluke-8200a-power-supply.kicad_pcb (KiCad board)
At the start: 2 copper layers, 229.2 x 79.4 mm, 77 parts, among them J10 Conn_01x01_Socket, J11 Conn_01x01_Socket, J12 Conn_01x01_Socket, J13 Conn_01x01_Socket, J14 Conn_01x01_Socket, J2 Conn_01x01_Socket, J3 Conn_01x01_Socket, J4 Conn_01x01_Socket, J5 Conn_01x01_Socket, J6 Conn_01x01_Socket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

Commit message: PCB quotable, but not yet fully compatable with fluke 8200A
Parts:
- D1, D2, D3, D4: value 1N5406 -> 1N5408
- D10: value 1N4001 -> 1N3068
- D5, D6, D7, D8: value 1N5406 -> 1N5404
- Q11: footprint Package_TO_SOT_THT:TO-3 -> TO-66:TO66
- moved D9 383.3 mm to (59.1, 84.5), turned to -90 degrees
- moved C13 380.0 mm to (62.9, 101.0), turned to -90 degrees
- moved D10 379.8 mm to (62.9, 84.5), turned to -90 degrees
- moved Q7 372.0 mm to (74.3, 97.5)
- moved Q5 364.6 mm to (75.6, 104.5)
- moved Q6 358.4 mm to (81.3, 97.5)
- moved Q4 350.8 mm to (82.5, 104.5)
- moved R7 172.4 mm to (69.8, 123.2), turned to 90 degrees
- moved R4 172.4 mm to (86.4, 123.2), turned to 90 degrees
- moved R6 169.8 mm to (78.7, 123.2), turned to 90 degrees
- moved R11 168.4 mm to (41.3, 97.2)
- moved R10 166.5 mm to (41.3, 88.3)
- moved R14 166.1 mm to (41.3, 101.6)
- moved R13 164.3 mm to (41.3, 92.7)
- moved R18 164.0 mm to (41.3, 106.0)
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Routing:
- net /+15V: track 0.00 -> 312.5 mm, vias 0 -> 4
- net /-15V: track 0.00 -> 262.0 mm, vias 0 -> 2
- net Net-(D6-K): track 0.00 -> 177.1 mm
- net Net-(D13-K): track 0.00 -> 172.1 mm
- net /+5V: track 0.00 -> 165.1 mm, vias 0 -> 2
- net Net-(D5-A): track 0.00 -> 164.1 mm, vias 0 -> 1
- net Net-(D2-K): track 0.00 -> 135.0 mm, vias 0 -> 1
- net Net-(D7-K): track 0.00 -> 101.1 mm
- net /+200V: track 0.00 -> 97.2 mm, vias 0 -> 2
- net Net-(D5-K): track 0.00 -> 88.4 mm
- net GNDS: track 0.00 -> 77.3 mm, vias 0 -> 4
- net Net-(D14-A): track 0.00 -> 73.4 mm
- net Net-(D13-A): track 0.00 -> 71.5 mm
- net Net-(D1-K): track 0.00 -> 69.5 mm
- net Net-(D3-K): track 0.00 -> 67.6 mm
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- added copper zone on B.Cu, net GND
- added copper zone on F.Cu, net GNDS
Other:
- outline, holes or cut-outs redrawn
