File: electronics/monostable-multivibrator/monostable-multivibrator.kicad_pcb (KiCad board)
At the start: 2 copper layers, 1 part, among them U1 NE555P

Commit message: footprints
Parts:
- added C1: C, Capacitor_THT:CP_Radial_D8.0mm_P3.80mm, F.Cu at (139.2, 37.1)
- added C2: 10nF, Capacitor_THT:C_Disc_D3.0mm_W1.6mm_P2.50mm, F.Cu at (139.2, 46.7)
- added C3: 0.33uF, Capacitor_THT:C_Disc_D3.0mm_W1.6mm_P2.50mm, F.Cu at (139.2, 56.2)
- added C4: 0.1uF, Capacitor_THT:C_Disc_D3.0mm_W1.6mm_P2.50mm, F.Cu at (139.2, 65.8)
- added D1: 1N4001, Diode_THT:D_DO-41_SOD81_P10.16mm_Horizontal, F.Cu at (147.8, 50.7)
- added D2: 1N4001, Diode_THT:D_DO-41_SOD81_P10.16mm_Horizontal, F.Cu at (147.8, 54.9)
- added J1: VCC_IN, Connector_PinHeader_1.00mm:PinHeader_1x01_P1.00mm_Horizontal, F.Cu at (147.4, 58.6)
- added J2: GND_IN, Connector_PinHeader_1.00mm:PinHeader_1x01_P1.00mm_Horizontal, F.Cu at (147.4, 61.6)
- added J3: LOAD_VIN, Connector_PinHeader_1.00mm:PinHeader_1x01_P1.00mm_Horizontal, F.Cu at (147.4, 64.7)
- added J4: LOAD_COM, Connector_PinHeader_1.00mm:PinHeader_1x01_P1.00mm_Horizontal, F.Cu at (147.4, 67.7)
- added JP1: Jumper_2_Open, Resistor_THT:R_Axial_DIN0207_L6.3mm_D2.5mm_P2.54mm_Vertical, F.Cu at (147.9, 34.4)
- added Q1: 2N2222, Package_TO_SOT_THT:TO-92, F.Cu at (153.7, 66.2)
- added R1: 100K, Resistor_THT:R_Axial_DIN0207_L6.3mm_D2.5mm_P2.54mm_Vertical, F.Cu at (147.9, 38.4)
- added R2: POT, Resistor_THT:R_Axial_DIN0207_L6.3mm_D2.5mm_P2.54mm_Vertical, F.Cu at (147.9, 42.5)
- added R3: 120, Resistor_THT:R_Axial_DIN0207_L6.3mm_D2.5mm_P2.54mm_Vertical, F.Cu at (147.9, 46.5)
- added SW1: SW_TRIG, Connector_PinHeader_1.00mm:PinHeader_1x03_P1.00mm_Horizontal, F.Cu at (154.8, 38.9)
- added SW2: SW_BYPASS, Connector_PinHeader_1.00mm:PinHeader_1x02_P1.00mm_Horizontal, F.Cu at (153.6, 33.9)
- added U2: LM7805_TO220, Package_TO_SOT_THT:TO-220-3_Vertical, F.Cu at (154.9, 61.0)
Connections:
- U1 pad 1: unconnected-(U1-GND-Pad1) -> GND
- U1 pad 2: unconnected-(U1-TR-Pad2) -> Net-(SW1-B)
- U1 pad 3: unconnected-(U1-Q-Pad3) -> /555_OUT
- U1 pad 4: unconnected-(U1-R-Pad4) -> /555_VIN
- U1 pad 5: unconnected-(U1-CV-Pad5) -> Net-(U1-CV)
- U1 pad 6: unconnected-(U1-THR-Pad6) -> Net-(U1-DIS)
- U1 pad 7: unconnected-(U1-DIS-Pad7) -> Net-(U1-DIS)
- U1 pad 8: unconnected-(U1-VCC-Pad8) -> /555_VIN

Commit message: looking finished
Parts:
- added H2: MountingHole_Pad, MountingHole:MountingHole_3.2mm_M3_DIN965_Pad_TopBottom, F.Cu at (167.6, 48.3)
- added H3: MountingHole_Pad, MountingHole:MountingHole_3.2mm_M3_DIN965_Pad_TopBottom, F.Cu at (127.0, 48.3)
- J1, J2, J3, J4: footprint Connector_PinHeader_1.00mm:PinHeader_1x01_P1.00mm_Horizontal -> Connector_PinHeader_2.00mm:PinHeader_1x01_P2.00mm_Vertical
- Q1: value 2N2222 -> 2N3904
- R1, R2, R3: footprint Resistor_THT:R_Axial_DIN0207_L6.3mm_D2.5mm_P2.54mm_Vertical -> Resistor_THT:R_Axial_DIN0207_L6.3mm_D2.5mm_P7.62mm_Horizontal
- SW1: footprint Connector_PinHeader_1.00mm:PinHeader_1x03_P1.00mm_Horizontal -> Connector_PinHeader_2.00mm:PinHeader_1x03_P2.00mm_Vertical
- SW2: footprint Connector_PinHeader_1.00mm:PinHeader_1x02_P1.00mm_Horizontal -> Connector_PinHeader_2.00mm:PinHeader_1x02_P2.00mm_Vertical
- moved SW2 46.7 mm to (140.7, 78.7), turned to -90 degrees
- moved C1 45.5 mm to (166.4, 73.7), turned to 180 degrees
- moved SW1 44.7 mm to (134.6, 78.7), turned to -90 degrees
- moved U1 32.4 mm to (156.2, 54.6)
- moved C2 30.3 mm to (162.6, 66.0)
- moved JP1 28.8 mm to (132.1, 58.4), turned to -90 degrees
- moved D1 27.8 mm to (132.1, 73.7)
- moved R1 22.6 mm to (146.1, 61.0)
- moved R2 22.5 mm to (167.6, 53.3), turned to -90 degrees
- moved D2 20.8 mm to (132.1, 68.6)
- moved R3 19.6 mm to (146.1, 66.0)
- moved U2 17.8 mm to (137.2, 61.0)
- moved J1 14.5 mm to (137.2, 48.3), turned to 180 degrees
- moved J2 14.3 mm to (142.2, 48.3), turned to 180 degrees
- moved J3 14.3 mm to (149.9, 78.7)
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Connections:
- D1 pad 1: Net-(D1-K) -> VCC
- D1 pad 2: GND -> Net-(D1-A)
- J4 pad 1: Net-(D1-K) -> Net-(D1-A)
- Q1 pad 1: Net-(D1-K) -> GND
- Q1 pad 3: GND -> Net-(D1-A)
Routing:
- net VCC: track 0.00 -> 67.3 mm
- net Net-(SW1-B): track 0.00 -> 51.2 mm
- net Net-(SW1-A): track 0.00 -> 41.0 mm
- net Net-(D2-K): track 0.00 -> 35.6 mm
- net Net-(U1-DIS): track 0.00 -> 20.1 mm
- net /555_OUT: track 0.00 -> 19.6 mm
- net Net-(D1-A): track 0.00 -> 13.3 mm
- net /555_VIN: track 0.00 -> 9.42 mm
- net Net-(Q1-B): track 0.00 -> 7.40 mm
- net Net-(U1-CV): track 0.00 -> 4.34 mm
- added copper zone on F.Cu, net /555_VIN
- added copper zone on B.Cu, net GND
Other:
- board outline added: 50.8 x 40.6 mm

Commit message: nice silkscreen updates
Parts:
- removed J3: LOAD_VIN, Connector_PinHeader_2.00mm:PinHeader_1x01_P2.00mm_Vertical
- removed J4: LOAD_COM, Connector_PinHeader_2.00mm:PinHeader_1x01_P2.00mm_Vertical
- C2, C3, C4: footprint Capacitor_THT:C_Disc_D3.0mm_W1.6mm_P2.50mm -> Capacitor_THT:C_Disc_D4.3mm_W1.9mm_P5.00mm
- J1: value VCC_IN -> + PWR -; footprint Connector_PinHeader_2.00mm:PinHeader_1x01_P2.00mm_Vertical -> Connector_PinSocket_2.54mm:PinSocket_1x02_P2.54mm_Vertical
- J2: value GND_IN -> - LOAD +; footprint Connector_PinHeader_2.00mm:PinHeader_1x01_P2.00mm_Vertical -> Connector_PinSocket_2.54mm:PinSocket_1x02_P2.54mm_Vertical
- SW1: value SW_TRIG -> CO NO NC
- SW2: value SW_BYPASS -> HOLD
- U2: value LM7805_TO220 -> LM7805
- moved J2 30.9 mm to (147.3, 78.7), turned to -90 degrees
- moved SW1 4.99 mm to (129.6, 78.7)
- moved SW2 3.81 mm to (136.9, 78.7)
- moved J1 2.52 mm to (134.6, 48.3), turned to 90 degrees
Connections:
- D1 pad 2: Net-(D1-A) -> /LOAD_COM
- J2 pad 1: GND -> VCC
- Q1 pad 3: Net-(D1-A) -> /LOAD_COM
Routing:
- net Net-(D1-A): track 13.3 -> 0.00 mm
- net /LOAD_COM: track 0.00 -> 13.3 mm
- net Net-(SW1-B): track 51.2 -> 57.6 mm
- net Net-(SW1-A): track 41.0 -> 47.1 mm
- net VCC: track 67.3 -> 63.7 mm
- net Net-(U1-DIS): track 20.1 -> 21.1 mm
- net Net-(U1-CV): track 4.34 -> 5.34 mm
- net Net-(D2-K): track 35.6 -> 36.5 mm
Other:
- board text added: "KEYS 2023 MONOSTABLE MULTIVIBRATOR"
- board text added: "SHORT JP1 TO BYPASS REG"
- board text added: "T = 1.1 * C1 * R2"

Commit message: added cap to fix repeated triggers
Parts:
- added C5: 100nF, Capacitor_THT:C_Disc_D4.3mm_W1.9mm_P5.00mm, F.Cu at (158.0, 75.7)
- SW2: value HOLD -> + -
Connections:
- U1 pad 2: Net-(SW1-B) -> Net-(U1-TR)
Routing:
- net Net-(SW1-B): track 57.6 -> 30.2 mm
- net Net-(U1-TR): track 0.00 -> 22.5 mm
Changed lines of the file:
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@@
   (net 10 "Net-(SW1-B)")
   (net 11 "/LOAD_COM")
+  (net 12 "Net-(U1-TR)")
   (footprint "Package_TO_SOT_THT:TO-92" (layer "F.Cu")
     (at 149.86 71.12 -90)
@@
     (property "ki_keywords" "NPN Transistor")
     (attr through_hole)
-    (fp_text reference "Q1" (at -0.635 -3.56) (layer "F.Fab")
-        (effects (font (size 1 1) (thickness 0.15)))
-    )
-    (fp_text value "2N3904" (at 1.27 -5.715 -180) (layer "F.SilkS")
+    (fp_text reference "Q1" (at -0.635 -3.56) (layer "F.SilkS")
+        (effects (font (size 1 1) (thickness 0.15)))
+    )
+    (fp_text value "2N3904" (at 1.27 -5.715) (layer "F.SilkS")
         (effects (font (size 1 1) (thickness 0.15)))
     )
@@
         (effects (font (size 1 1) (thickness 0.15)))
     )
-    (fp_text value "HOLD" (at 2.54 1) (layer "F.SilkS")
+    (fp_text value "+ -" (at 2.54 1) (layer "F.SilkS")
         (effects (font (size 1 1) (thickness 0.15)))
     )
@@
     )
   )
+  (footprint "Capacitor_THT:C_Disc_D4.3mm_W1.9mm_P5.00mm" (layer "F.Cu")
+    (at 157.977767 75.702233 -135)
+    (descr "C, Disc series, Radial, pin pitch=5.00mm, , diameter*width=4.3*1.9mm^2, Capacitor, http://www.vishay.com/docs/45233/krseries.pdf")
+    (tags "C Disc series Radial pin pitch 5.00mm  diameter 4.3mm width 1.9mm Capacitor")
+    (property "Sheetfile" "monostable-multivibrator.kicad_sch")
+    (property "Sheetname" "")
+    (property "ki_description" "Unpolarized capacitor")
+    (property "ki_keywords" "cap capacitor")
+    (attr through_hole)
+    (fp_text reference "C5" (at 2.949013 2.245064 45) (layer "F.SilkS")
+        (effects (font (size 1 1) (thickness 0.15)))
+    )
+    (fp_text value "100nF" (at 2.050987 -2.245064 45) (layer "F.SilkS")
+        (effects (font (size 1 1) (thickness 0.15)))
+    )
+    (fp_text user "${REFERENCE}" (at 2.5 0 45) (layer "F.Fab")
+        (effects (font (size 0.86 0.86) (thickness 0.129)))
+    )
+    (fp_line (start 0.23 -1.07) (end 0.23 -1.055)
+      (stroke (width 0.12) (type solid)) (layer "F.SilkS"))
+    (fp_line (start 0.23 -1.07) (end 4.77 -1.07)
+      (stroke (width 0.12) (type solid)) (layer "F.SilkS"))
+    (fp_line (start 0.23 1.055) (end 0.23 1.07)
+      (stroke (width 0.12) (type solid)) (layer "F.SilkS"))
+    (fp_line (start 0.23 1.07) (end 4.77 1.07)
+      (stroke (width 0.12) (type solid)) (layer "F.SilkS"))
+    (fp_line (start 4.77 -1.07) (end 4.77 -1.055)
+      (stroke (width 0.12) (type solid)) (layer "F.SilkS"))
+    (fp_line (start 4.77 1.055) (end 4.77 1.07)
+      (stroke (width 0.12) (type solid)) (layer "F.SilkS"))
+    (fp_line (start -1.05 -1.2) (end -1.05 1.2)
+      (stroke (width 0.05) (type solid)) (layer "F.CrtYd"))
+    (fp_line (start -1.05 1.2) (end 6.05 1.2)
+      (stroke (width 0.05) (type solid)) (layer "F.CrtYd"))
+    (fp_line (start 6.05 -1.2) (end -1.05 -1.2)
+      (stroke (width 0.05) (type solid)) (layer "F.CrtYd"))
+    (fp_line (start 6.05 1.2) (end 6.05 -1.2)
+      (stroke (width 0.05) (type solid)) (layer "F.CrtYd"))
+    (fp_line (start 0.35 -0.95) (end 0.35 0.95)
+      (stroke (width 0.1) (type solid)) (layer "F.Fab"))
+    (fp_line (start 0.35 0.95) (end 4.65 0.95)
+      (stroke (width 0.1) (type solid)) (layer "F.Fab"))
+    (fp_line (start 4.65 -0.95) (end 0.35 -0.95)
+      (stroke (width 0.1) (type solid)) (layer "F.Fab"))
+    (fp_line (start 4.65 0.95) (end 4.65 -0.95)
+      (stroke (width 0.1) (type solid)) (layer "F.Fab"))
+    (pad "1" thru_hole circle (at 0 0 225) (size 1.6 1.6) (drill 0.8) (layers "*.Cu" "*.Mask")
+      (net 12 "Net-(U1-TR)") (pintype "passive"))
+    (pad "2" thru_hole circle (at 5 0 225) (size 1.6 1.6) (drill 0.8) (layers "*.Cu" "*.Mask")
+      (net 10 "Net-(SW1-B)") (pintype "passive"))
+    (model "${KICAD6_3DMODEL_DIR}/Capacitor_THT.3dshapes/C_Disc_D4.3mm_W1.9mm_P5.00mm.wrl"
+      (offset (xyz 0 0 0))
+      (scale (xyz 1 1 1))
+      (rotate (xyz 0 0 0))
+    )
+  )
   (footprint "Package_DIP:DIP-8_W7.62mm" (layer "F.Cu")
     (at 156.22 54.62)
@@
       (net 2 "GND") (pinfunction "GND") (pintype "power_in"))
     (pad "2" thru_hole oval (at 0 2.54) (size 1.6 1.6) (drill 0.8) (layers "*.Cu" "*.Mask")
-      (net 10 "Net-(SW1-B)") (pinfunction "TR") (pintype "input"))
+      (net 12 "Net-(U1-TR)") (pinfunction "TR") (pintype "input"))
     (pad "3" thru_hole oval (at 0 5.08) (size 1.6 1.6) (drill 0.8) (layers "*.Cu" "*.Mask")
       (net 7 "/555_OUT") (pinfunction "Q") (pintype "output"))
@@
   (segment (start 129.635 78.74) (end 129.635 80.74) (width 0.25) (layer "B.Cu") (net 9))
   (segment (start 127.635 81.28) (end 127.635 78.74) (width 0.25) (layer "B.Cu") (net 10))
-  (segment (start 158.76 57.16) (end 156.22 57.16) (width 0.25) (layer "B.Cu") (net 10))
-  (segment (start 160.02 58.42) (end 158.76 57.16) (width 0.25) (layer "B.Cu") (net 10))
-  (segment (start 152.4 81.28) (end 160.02 73.66) (width 0.25) (layer "B.Cu") (net 10))
   (segment (start 127.635 81.28) (end 152.4 81.28) (width 0.25) (layer "B.Cu") (net 10))
-  (segment (start 160.02 73.66) (end 160.02 58.42) (width 0.25) (layer "B.Cu") (net 10))
+  (segment (start 152.4 81.28) (end 154.442233 79.237767) (width 0.25) (layer "B.Cu") (net 10))
   (segment (start 149.86 73.66) (end 144.78 78.74) (width 1) (layer "F.Cu") (net 11))
   (segment (start 142.24 76.2) (end 144.78 78.74) (width 0.5) (layer "F.Cu") (net 11))
   (segment (start 142.24 73.66) (end 142.24 76.2) (width 0.5) (layer "F.Cu") (net 11))
+  (segment (start 158.76 57.16) (end 156.22 57.16) (width 0.25) (layer "B.Cu") (net 12))
+  (segment (start 160.02 58.42) (end 158.76 57.16) (width 0.25) (layer "B.Cu") (net 12))
+  (segment (start 157.977767 75.702233) (end 160.02 73.66) (width 0.25) (layer "B.Cu") (net 12))
+  (segment (start 160.02 73.66) (end 160.02 58.42) (width 0.25) (layer "B.Cu") (net 12))
   (zone (net 5) (net_name "/555_VIN") (layer "F.Cu") (hatch edge 0.5)
     (connect_pads (clearance 0.5))

Commit message: bug fix, held button should no longer keep switch active.
Parts:
- SW1: value CO NO NC -> NO CO NC
Connections:
- R1 pad 2: Net-(SW1-A) -> Net-(U1-TR)
- SW1 pad 1: Net-(SW1-A) -> /555_VIN
Routing:
- net Net-(SW1-A): track 47.1 -> 0.00 mm
- net /LOAD_COM: track 13.3 -> 14.8 mm
- net Net-(U1-TR): track 22.5 -> 21.4 mm
Changed lines of the file:
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@@
   (net 7 "/555_OUT")
   (net 8 "Net-(Q1-B)")
-  (net 9 "Net-(SW1-A)")
-  (net 10 "Net-(SW1-B)")
-  (net 11 "/LOAD_COM")
-  (net 12 "Net-(U1-TR)")
+  (net 9 "Net-(SW1-B)")
+  (net 10 "/LOAD_COM")
+  (net 11 "Net-(U1-TR)")
   (footprint "Package_TO_SOT_THT:TO-92" (layer "F.Cu")
     (at 149.86 71.12 -90)
@@
       (net 8 "Net-(Q1-B)") (pinfunction "B") (pintype "passive"))
     (pad "3" thru_hole circle (at 2.54 0 270) (size 1.3 1.3) (drill 0.75) (layers "*.Cu" "*.Mask")
-      (net 11 "/LOAD_COM") (pinfunction "C") (pintype "passive"))
+      (net 10 "/LOAD_COM") (pinfunction "C") (pintype "passive"))
     (model "${KICAD6_3DMODEL_DIR}/Package_TO_SOT_THT.3dshapes/TO-92.wrl"
       (offset (xyz 0 0 0))
@@
       (net 5 "/555_VIN") (pintype "passive"))
     (pad "2" thru_hole oval (at 7.62 0) (size 1.6 1.6) (drill 0.8) (layers "*.Cu" "*.Mask")
-      (net 9 "Net-(SW1-A)") (pintype "passive"))
+      (net 11 "Net-(U1-TR)") (pintype "passive"))
     (model "${KICAD6_3DMODEL_DIR}/Resistor_THT.3dshapes/R_Axial_DIN0207_L6.3mm_D2.5mm_P7.62mm_Horizontal.wrl"
       (offset (xyz 0 0 0))
@@
         (effects (font (size 1 1) (thickness 0.15)))
     )
-    (fp_text value "CO NO NC" (at 2.54 2 180) (layer "F.SilkS")
+    (fp_text value "NO CO NC" (at 2.54 2 180) (layer "F.SilkS")
         (effects (font (size 1 1) (thickness 0.15)))
     )
@@
       (stroke (width 0.1) (type solid)) (layer "F.Fab"))
     (pad "1" thru_hole rect (at 0 0 270) (size 1.35 1.35) (drill 0.8) (layers "*.Cu" "*.Mask")
-      (net 9 "Net-(SW1-A)") (pinfunction "A") (pintype "passive"))
+      (net 5 "/555_VIN") (pinfunction "A") (pintype "passive"))
     (pad "2" thru_hole oval (at 0 2 270) (size 1.35 1.35) (drill 0.8) (layers "*.Cu" "*.Mask")
-      (net 10 "Net-(SW1-B)") (pinfunction "B") (pintype "passive"))
+      (net 9 "Net-(SW1-B)") (pinfunction "B") (pintype "passive"))
     (pad "3" thru_hole oval (at 0 4 270) (size 1.35 1.35) (drill 0.8) (layers "*.Cu" "*.Mask")
       (net 2 "GND") (pinfunction "C") (pintype "passive"))
@@
       (stroke (width 0.1) (type solid)) (layer "F.Fab"))
     (pad "1" thru_hole circle (at 0 0 225) (size 1.6 1.6) (drill 0.8) (layers "*.Cu" "*.Mask")
-      (net 12 "Net-(U1-TR)") (pintype "passive"))
+      (net 11 "Net-(U1-TR)") (pintype "passive"))
     (pad "2" thru_hole circle (at 5 0 225) (size 1.6 1.6) (drill 0.8) (layers "*.Cu" "*.Mask")
-      (net 10 "Net-(SW1-B)") (pintype "passive"))
+      (net 9 "Net-(SW1-B)") (pintype "passive"))
     (model "${KICAD6_3DMODEL_DIR}/Capacitor_THT.3dshapes/C_Disc_D4.3mm_W1.9mm_P5.00mm.wrl"
       (offset (xyz 0 0 0))
@@
       (net 2 "GND") (pinfunction "GND") (pintype "power_in"))
     (pad "2" thru_hole oval (at 0 2.54) (size 1.6 1.6) (drill 0.8) (layers "*.Cu" "*.Mask")
-      (net 12 "Net-(U1-TR)") (pinfunction "TR") (pintype "input"))
+      (net 11 "Net-(U1-TR)") (pinfunction "TR") (pintype "input"))
     (pad "3" thru_hole oval (at 0 5.08) (size 1.6 1.6) (drill 0.8) (layers "*.Cu" "*.Mask")
       (net 7 "/555_OUT") (pinfunction "Q") (pintype "output"))
@@
       (net 4 "VCC") (pinfunction "Pin_1") (pintype "passive"))
     (pad "2" thru_hole oval (at 0 2.54 270) (size 1.7 1.7) (drill 1) (layers "*.Cu" "*.Mask")
-      (net 11 "/LOAD_COM") (pinfunction "Pin_2") (pintype "passive"))
+      (net 10 "/LOAD_COM") (pinfunction "Pin_2") (pintype "passive"))
     (model "${KICAD6_3DMODEL_DIR}/Connector_PinSocket_2.54mm.3dshapes/PinSocket_1x02_P2.54mm_Vertical.wrl"
       (offset (xyz 0 0 0))
@@
       (net 4 "VCC") (pinfunction "K") (pintype "passive"))
     (pad "2" thru_hole oval (at 10.16 0) (size 2.2 2.2) (drill 1.1) (layers "*.Cu" "*.Mask")
-      (net 11 "/LOAD_COM") (pinfunction "A") (pintype "passive"))
+      (net 10 "/LOAD_COM") (pinfunction "A") (pintype "passive"))
     (model "${KICAD6_3DMODEL_DIR}/Diode_THT.3dshapes/D_DO-41_SOD81_P10.16mm_Horizontal.wrl"
       (offset (xyz 0 0 0))
@@
   (segment (start 151.13 72.39) (end 151.13 68.58) (width 0.25) (layer "F.Cu") (net 8))
   (segment (start 151.13 68.58) (end 153.67 66.04) (width 0.25) (layer "F.Cu") (net 8))
-  (segment (start 157.48 73.66) (end 157.48 66.04) (width 0.25) (layer "B.Cu") (net 9))
-  (segment (start 150.31 80.83) (end 157.48 73.66) (width 0.25) (layer "B.Cu") (net 9))
-  (segment (start 129.635 80.74) (end 129.725 80.83) (width 0.25) (layer "B.Cu") (net 9))
-  (segment (start 157.48 66.04) (end 153.67 62.23) (width 0.25) (layer "B.Cu") (net 9))
-  (segment (start 153.67 62.23) (end 153.67 60.96) (width 0.25) (layer "B.Cu") (net 9))
-  (segment (start 129.725 80.83) (end 150.31 80.83) (width 0.25) (layer "B.Cu") (net 9))
-  (segment (start 129.635 78.74) (end 129.635 80.74) (width 0.25) (layer "B.Cu") (net 9))
-  (segment (start 127.635 81.28) (end 127.635 78.74) (width 0.25) (layer "B.Cu") (net 10))
-  (segment (start 127.635 81.28) (end 152.4 81.28) (width 0.25) (layer "B.Cu") (net 10))
-  (segment (start 152.4 81.28) (end 154.442233 79.237767) (width 0.25) (layer "B.Cu") (net 10))
-  (segment (start 149.86 73.66) (end 144.78 78.74) (width 1) (layer "F.Cu") (net 11))
-  (segment (start 142.24 76.2) (end 144.78 78.74) (width 0.5) (layer "F.Cu") (net 11))
-  (segment (start 142.24 73.66) (end 142.24 76.2) (width 0.5) (layer "F.Cu") (net 11))
-  (segment (start 158.76 57.16) (end 156.22 57.16) (width 0.25) (layer "B.Cu") (net 12))
-  (segment (start 160.02 58.42) (end 158.76 57.16) (width 0.25) (layer "B.Cu") (net 12))
-  (segment (start 157.977767 75.702233) (end 160.02 73.66) (width 0.25) (layer "B.Cu") (net 12))
-  (segment (start 160.02 73.66) (end 160.02 58.42) (width 0.25) (layer "B.Cu") (net 12))
+  (segment (start 127.635 81.28) (end 127.635 78.74) (width 0.25) (layer "F.Cu") (net 9))
+  (segment (start 152.4 81.28) (end 127.635 81.28) (width 0.25) (layer "F.Cu") (net 9))
+  (segment (start 154.442233 79.237767) (end 152.4 81.28) (width 0.25) (layer "F.Cu") (net 9))
+  (segment (start 144.78 76.2) (end 144.78 78.74) (width 1) (layer "F.Cu") (net 10))
+  (segment (start 142.24 76.2) (end 144.78 78.74) (width 0.5) (layer "F.Cu") (net 10))
+  (segment (start 147.32 76.2) (end 144.78 76.2) (width 1) (layer "F.Cu") (net 10))
+  (segment (start 149.86 73.66) (end 147.32 76.2) (width 1) (layer "F.Cu") (net 10))
+  (segment (start 142.24 73.66) (end 142.24 76.2) (width 0.5) (layer "F.Cu") (net 10))
+  (segment (start 153.67 60.96) (end 153.67 59.71) (width 0.25) (layer "F.Cu") (net 11))
+  (segment (start 153.67 62.23) (end 153.67 60.96) (width 0.25) (layer "F.Cu") (net 11))
+  (segment (start 153.67 59.71) (end 156.22 57.16) (width 0.25) (layer "F.Cu") (net 11))
+  (segment (start 157.977767 75.702233) (end 157.977767 66.537767) (width 0.25) (layer "F.Cu") (net 11))
+  (segment (start 157.977767 66.537767) (end 153.67 62.23) (width 0.25) (layer "F.Cu") (net 11))
   (zone (net 5) (net_name "/555_VIN") (layer "F.Cu") (hatch edge 0.5)
     (connect_pads (clearance 0.5))
